File: PCB/audio-receiver/amp-channel.kicad_sch (KiCad schematic)
At the start: 36 parts, among them Q1 BC559, Q2 BC639, Q3 BC639, Q4 BC640, Q5 MJE3055, Q6 MJE2955

Commit message: update schematic and start work on BOM
Parts:
- removed F1: 1A, symbol Device:Fuse
- C1: Mouser URL (none) -> https://www.mouser.com/ProductDetail/Wurth-Elektronik/86002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
- C2, C4, C8: Mouser URL (none) -> https://www.mouser.com/ProductDetail/Nichicon/UVR1H101MPD1T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
- C3: Mouser URL (none) -> https://www.mouser.com/ProductDetail/Walsin/YP501101K040BAN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
- C5: Mouser URL (none) -> https://www.mouser.com/ProductDetail/Rubycon/35YXJ2200M16X2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
- C6: Mouser URL (none) -> https://www.mouser.com/ProductDetail/Wurth-Elektronik/86001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
- C7: Mouser URL (none) -> https://www.mouser.com/ProductDetail/Walsin/YV101103Z060HAN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
- D1, D2, D3, D4: Mouser URL (none) -> https://www.mouser.com/ProductDetail/onsemi-Fairchild/1N414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
- D5, D6, D7, D8: Mouser URL (none) -> https://www.mouser.com/ProductDetail/Diotec-Semiconductor/U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
- Q1: footprint Package_TO_SOT_THT:TO-92_Inline -> (none); Mouser URL (none) -> https://www.mouser.com/ProductDetail/Diotec-Semiconductor/B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
- Q2, Q3: Mouser URL (none) -> https://www.mouser.com/ProductDetail/onsemi-Fairchild/BC639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
Connections:
- net VCC: now also C8.1, Q3.C, Q5.C, R11.2, R6.1

Commit message: add bom, edit symbols, assign some footprints
Parts:
- removed Q2, Q3: BC639, symbol Device:Q_NPN
- removed Q4: BC640, symbol Device:Q_PNP
- added Q2, Q3: BD139, Package_TO_SOT_THT:TO-126-3_Vertical, symbol Transistor_BJT:BD139
- added Q4: BD140, Package_TO_SOT_THT:TO-126-3_Vertical, symbol Transistor_BJT:BD140
- C1: footprint (none) -> Capacitor_THT:CP_Radial_D5.0mm_P2.00mm; Mouser PN (none) -> 710-860020672010
- C2, C4, C8: footprint (none) -> Capacitor_THT:CP_Radial_D8.0mm_P3.50mm; Mouser PN (none) -> 647-UVR1H101MPD1TD
- C3: footprint (none) -> Capacitor_THT:C_Disc_D4.3mm_W1.9mm_P5.00mm; Mouser PN (none) -> 791-YP501101K40AND5
- C5: footprint (none) -> Capacitor_THT:CP_Radial_D16.0mm_P7.50mm; Mouser PN (none) -> 232-35YXJ2200M16X25
- C6: footprint (none) -> Capacitor_THT:CP_Radial_D5.0mm_P2.00mm; Mouser PN (none) -> 710-860010672011
- C7: footprint (none) -> Capacitor_THT:C_Disc_D4.3mm_W1.9mm_P5.00mm; Mouser PN (none) -> 791-YV101103Z60HAND5
- D1, D2, D3, D4: footprint (none) -> Diode_THT:D_DO-35_SOD27_P7.62mm_Horizontal; Mouser PN (none) -> 512-1N4148T50R
- D5, D6, D7, D8: footprint (none) -> Diode_THT:D_DO-41_SOD81_P7.62mm_Horizontal; Mouser PN (none) -> 637-UF4004
- Q1: footprint (none) -> Package_TO_SOT_THT:TO-92_Inline_Wide; Mouser PN (none) -> 637-BC559A
- Q5: footprint (none) -> Package_TO_SOT_THT:TO-220-3_Vertical; Mouser PN (none) -> 863-MJE3055TG; Mouser URL (none) -> https://www.mouser.com/ProductDetail/onsemi/MJE3055TG?qs=HV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
- Q6: footprint (none) -> Package_TO_SOT_THT:TO-220-3_Vertical; Mouser PN (none) -> 863-MJE2955TG; Mouser URL (none) -> https://www.mouser.com/ProductDetail/onsemi/MJE2955TG?qs=HV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
- R1, R2: Mouser PN (none) -> 603-MFR-25FTF52-33K; Mouser URL (none) -> https://www.mouser.com/ProductDetail/YAGEO/MFR-25FTF52-33K?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
- R10, R9: Mouser PN (none) -> 603-SQP500JB-2R7; Mouser URL (none) -> https://www.mouser.com/ProductDetail/YAGEO/SQP500JB-2R7?qs=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
- R11: Mouser PN (none) -> 603-MFR25SFTF26-12K; Mouser URL (none) -> https://www.mouser.com/ProductDetail/YAGEO/MFR25SFTF26-12K?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
- R12, R3, R6, R7: Mouser PN (none) -> 603-MF0207FTE52-2K2; Mouser URL (none) -> https://www.mouser.com/ProductDetail/YAGEO/MF0207FTE52-2K2?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
- R13: Mouser PN (none) -> 603-CFR-25JR-52-2R7; Mouser URL (none) -> https://www.mouser.com/ProductDetail/YAGEO/CFR-25JR-52-2R7?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
- R4: Mouser PN (none) -> 603-MFR-12FTF52-100R; Mouser URL (none) -> https://www.mouser.com/ProductDetail/YAGEO/MFR-12FTF52-100R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
- R5: Mouser PN (none) -> 603-MFR-25FTF52-1K; Mouser URL (none) -> https://www.mouser.com/ProductDetail/YAGEO/MFR-25FTF52-1K?q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
- R8: Mouser PN (none) -> 603-FMP200JR-52-560R; Mouser URL (none) -> https://www.mouser.com/ProductDetail/YAGEO/FMP200JR-52-560R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
Connections:
- net GND: now also Q6.2 (C), Q2.1 (E), Q4.2 (C); no longer Q6.C
- net VCC: now also Q5.2 (C), Q3.2 (C); no longer Q5.C
- net at D1.2 (A), R7.2: now also Q3.3 (B)
- net at R8.1: now also Q5.1 (B), Q3.1 (E); no longer Q5.B
- net at D6.1 (K), D8.1 (K), R10.2: now also Q6.3 (E); no longer Q6.E
- net at C3.2, D4.1 (K): now also Q2.2 (C), Q4.3 (B)
- net at D5.2 (A), D7.2 (A), R9.1: now also Q5.3 (E); no longer Q5.E
- net at C3.1, Q1.1 (C), R5.1: now also Q2.3 (B)
- net at R8.2: now also Q6.1 (B), Q4.1 (E); no longer Q6.B

Commit message: update pcb/bom and add new schematic for input board
Parts:
- R1, R11, R12, R13, R2, R3, R5, R6, R7: footprint (none) -> Resistor_THT:R_Axial_DIN0207_L6.3mm_D2.5mm_P7.62mm_Horizontal
- R10, R9: footprint (none) -> Resistor_THT:R_Axial_Power_L25.0mm_W9.0mm_P27.94mm
- R4: footprint (none) -> Resistor_THT:R_Axial_DIN0204_L3.6mm_D1.6mm_P5.08mm_Horizontal
- R8: footprint (none) -> Resistor_THT:R_Axial_DIN0309_L9.0mm_D3.2mm_P12.70mm_Horizontal
