File: PCB/control-board/control-board.kicad_sch (KiCad schematic)
At the start: 3 parts, among them J1 OLED, U1 ATtiny84A-SS

Commit message: update control board schematic s
Parts:
- added J2: PROGRAM, symbol Connector:Conn_01x04_Pin
- added SW1, SW2, SW3, SW4: SW_Push, symbol Switch:SW_Push
Connections:
- net GND: now also SW1.2, SW2.2, SW3.2, SW4.2
- net OLED_SCL: now also U1.12 (PA1)
- net OLED_SDA: now also U1.13 (AREF/PA0)
- net SW2: now reaches U1.10 (PA3)
- net SW2: now also SW2.1
- net SW1: now reaches U1.11 (PA2)
- net SW1: now also SW1.1
- net CTRL_A: now reaches U1.2 (XTAL1/PB0)
- net CTRL_B: now reaches U1.3 (XTAL2/PB1)
- net at U1.4 (~{RESET}/PB3): now also J2.1 (Pin_1)
- net MUTE: now reaches U1.5 (PB2)
- net at U1.7 (PA6): now also J2.2 (Pin_2)
- net SW4: now reaches U1.8 (PA5)
- net SW4: now also J2.3 (Pin_3), SW4.1
- net SW3: now reaches U1.9 (PA4)
- net SW3: now also J2.4 (Pin_4), SW3.1
- no-connect marks 0 -> 1
Other:
- moved on the sheet: J1

Commit message: bom, readme, cad, pcb
Parts:
- added J3: Screw_Terminal_01x04, Connector_Phoenix_MSTB:PhoenixContact_MSTBA_2,5_4-G-5,08_1x04_P5.08mm_Horizontal, symbol Connector:Screw_Terminal_01x04
- added J4: Screw_Terminal_01x02, TerminalBlock_CUI:TerminalBlock_CUI_TB007-508-02_1x02_P5.08mm_Horizontal, symbol Connector:Screw_Terminal_01x02
- added SW5: SW_Push, Button_Switch_THT:SW_PUSH_6mm, symbol Switch:SW_Push
- J1: footprint (none) -> KiCad-SSD1306-0.91-OLED-4pin-128x32:SSD1306-0.91-OLED-4pin-128x32; now not fitted; now left out of the parts list
- J2: footprint (none) -> Connector_PinHeader_2.54mm:PinHeader_1x04_P2.54mm_Vertical; now not fitted; now left out of the parts list
- SW1, SW2, SW3, SW4: footprint (none) -> Button_Switch_THT:SW_PUSH_6mm; Mouser PN (none) -> 179-TS026655BK260LCR
- U1: Mouser PN (none) -> 556-ATTINY84A-SSFR
Connections:
- net +5V: now also J4.1 (Pin_1)
- net CTRL_A: now also J3.1 (Pin_1)
- net CTRL_B: now also J3.2 (Pin_2)
- net GND: now also J3.4 (Pin_4), J4.2 (Pin_2), SW5.2
- net MUTE: now also J3.3 (Pin_3)
- net SW5: now reaches J2.2 (Pin_2), U1.7 (PA6)
- net SW5: now also SW5.1
Other:
- moved on the sheet: C1, SW1, SW2, SW3, SW4, U1
