File: PCB/control-board/control-board.kicad_pcb (KiCad board)
At the start: 2 copper layers, 91 x 56.5 mm, 11 parts, among them J1 OLED, J2 PROGRAM, J3 Screw_Terminal_01x04, J4 Screw_Terminal_01x02, SW1 SW_Push, SW2 SW_Push, SW3 SW_Push, SW4 SW_Push, SW5 SW_Push, U1 ATtiny84A-SS

Commit message: fix power supply on pcb
Routing:
- net GND: vias 0 -> 3
Other:
- board text added: "+5V GND"
Changed lines of the file:
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@@
 		(layer "Edge.Cuts")
+	)
+	(gr_text "+5V   GND"
+		(at 111.5 103 270)
+		(layer "B.SilkS")
+		(effects
+			(font
+				(size 1 1)
+				(thickness 0.1)
+			)
+			(justify left bottom mirror)
+		)
 	)
 	(segment
@@
 		(net 1)
 	)
+	(via
+		(at 131.5 75.5)
+		(size 0.6)
+		(drill 0.3)
+		(layers "F.Cu" "B.Cu")
+		(free yes)
+		(net 2)
+	)
+	(via
+		(at 130.5 75.5)
+		(size 0.6)
+		(drill 0.3)
+		(layers "F.Cu" "B.Cu")
+		(free yes)
+		(net 2)
+	)
+	(via
+		(at 132.5 75.5)
+		(size 0.6)
+		(drill 0.3)
+		(layers "F.Cu" "B.Cu")
+		(free yes)
+		(net 2)
+	)
 	(segment
